File: MonochromeVGA/MonochromeVGA.brd (EAGLE design)
At the start: 59.7 x 37.1 mm, 12 parts

Commit message: Add files via upload
Parts:
- 1R, 2G', 3B, 4G: device diode:DO35-7 -> diode:D-5
Connections:
- net 1R renamed N$6
- net 2G' renamed N$3
- net 3B renamed N$4
- net 4G renamed N$5
Routing:
- net N$6: track 0.00 -> 11.3 mm, vias 0 -> 1
- net N$3: track 0.00 -> 7.56 mm
- net N$5: track 0.00 -> 7.56 mm
- net N$4: track 0.00 -> 5.71 mm
- net LUMA: track 65.0 -> 62.8 mm
Changed lines of the file:
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@@
 <attribute name="HEIGHT" value="5mm" x="29.21" y="83.185" size="1.778" layer="27" rot="R180" display="off"/>
 </element>
-<element name="2G'" library="diode" package="DO35-7" value="" x="25.4" y="59.055"/>
-<element name="3B" library="diode" package="DO35-7" value="" x="32.385" y="59.055"/>
-<element name="4G" library="diode" package="DO35-7" value="" x="39.37" y="59.055"/>
-<element name="1R" library="diode" package="DO35-7" value="" x="18.415" y="59.055"/>
+<element name="2G'" library="diode" package="D-5" value="" x="25.4" y="59.055"/>
+<element name="3B" library="diode" package="D-5" value="" x="32.385" y="59.055"/>
+<element name="4G" library="diode" package="D-5" value="" x="39.37" y="59.055"/>
+<element name="1R" library="diode" package="D-5" value="" x="18.415" y="59.055"/>
 </elements>
 <signals>
@@
 <wire x1="30.1625" y1="77.31125" x2="38.89375" y2="77.31125" width="0.254" layer="1"/>
 <wire x1="30.1625" y1="77.31125" x2="30.083125" y2="77.231875" width="0.254" layer="1"/>
-<wire x1="22.06625" y1="60.16625" x2="22.225" y2="59.055" width="0.254" layer="1"/>
+<wire x1="22.06625" y1="60.16625" x2="20.955" y2="59.055" width="0.254" layer="1"/>
 <wire x1="26.82875" y1="60.16625" x2="22.06625" y2="60.16625" width="0.254" layer="1"/>
-<wire x1="29.21" y1="59.055" x2="26.908125" y2="60.086875" width="0.254" layer="1"/>
+<wire x1="27.94" y1="59.055" x2="26.908125" y2="60.086875" width="0.254" layer="1"/>
 <wire x1="26.908125" y1="60.086875" x2="26.82875" y2="60.16625" width="0.254" layer="1"/>
 <wire x1="33.81375" y1="60.16625" x2="33.893125" y2="60.086875" width="0.254" layer="1"/>
-<wire x1="33.893125" y1="60.086875" x2="36.195" y2="59.055" width="0.254" layer="1"/>
+<wire x1="33.893125" y1="60.086875" x2="34.925" y2="59.055" width="0.254" layer="1"/>
 <wire x1="26.9875" y1="60.16625" x2="33.81375" y2="60.16625" width="0.254" layer="1"/>
 <wire x1="26.9875" y1="60.16625" x2="26.908125" y2="60.086875" width="0.254" layer="1"/>
-<wire x1="40.79875" y1="60.16625" x2="43.18" y2="59.055" width="0.254" layer="1"/>
+<wire x1="40.79875" y1="60.16625" x2="41.91" y2="59.055" width="0.254" layer="1"/>
 <wire x1="33.9725" y1="60.16625" x2="40.79875" y2="60.16625" width="0.254" layer="1"/>
 <wire x1="33.9725" y1="60.16625" x2="33.893125" y2="60.086875" width="0.254" layer="1"/>
 <wire x1="22.225" y1="60.325" x2="22.225" y2="76.2" width="0.254" layer="16"/>
-<wire x1="22.225" y1="59.055" x2="22.225" y2="60.325" width="0.254" layer="16"/>
+<wire x1="20.955" y1="59.055" x2="22.225" y2="60.325" width="0.254" layer="16"/>
 </signal>
 <signal name="R_OUT">
@@
 <signal name="N$1">
 </signal>
-<signal name="1R">
+<signal name="N$3">
+<contactref element="2G'" pad="C"/>
+<contactref element="SW1" pad="2"/>
+<wire x1="22.86" y1="60.325" x2="22.86" y2="59.055" width="0.254" layer="16"/>
+<wire x1="27.305" y1="64.77" x2="22.86" y2="60.325" width="0.254" layer="16"/>
+</signal>
+<signal name="N$4">
+<contactref element="3B" pad="C"/>
+<contactref element="SW1" pad="3"/>
+<wire x1="29.845" y1="64.77" x2="29.845" y2="59.055" width="0.254" layer="16"/>
+</signal>
+<signal name="N$5">
+<contactref element="4G" pad="C"/>
+<contactref element="SW1" pad="4"/>
+<wire x1="32.385" y1="63.5" x2="32.385" y2="64.77" width="0.254" layer="16"/>
+<wire x1="36.83" y1="59.055" x2="32.385" y2="63.5" width="0.254" layer="16"/>
+</signal>
+<signal name="N$6">
 <contactref element="1R" pad="C"/>
 <contactref element="SW1" pad="1"/>
-<wire x1="14.605" y1="59.055" x2="24.765" y2="64.77" width="0" layer="19" extent="1-1"/>
-</signal>
-<signal name="2G'">
-<contactref element="2G'" pad="C"/>
-<contactref element="SW1" pad="2"/>
-<wire x1="21.59" y1="59.055" x2="27.305" y2="64.77" width="0" layer="19" extent="1-1"/>
-</signal>
-<signal name="3B">
-<contactref element="3B" pad="C"/>
-<contactref element="SW1" pad="3"/>
-<wire x1="28.575" y1="59.055" x2="29.845" y2="64.77" width="0" layer="19" extent="1-1"/>
-</signal>
-<signal name="4G">
-<contactref element="4G" pad="C"/>
-<contactref element="SW1" pad="4"/>
-<wire x1="32.385" y1="64.77" x2="35.56" y2="59.055" width="0" layer="19" extent="1-1"/>
+<wire x1="21.2725" y1="64.4525" x2="15.875" y2="59.055" width="0.254" layer="16"/>
+<wire x1="21.59" y1="64.77" x2="21.2725" y2="64.4525" width="0.254" layer="1"/>
+<wire x1="24.765" y1="64.77" x2="21.59" y2="64.77" width="0.254" layer="1"/>
+<via x="21.2725" y="64.4525" extent="1-16" drill="0.6096"/>
 </signal>
 </signals>
